File: Indosluch_AM/Indosluch_AM/Indosluch_AM_modules_round.kicad_pcb (KiCad board)
At the start: 2 copper layers, 40 parts, among them J1 Con1x03, J2 Con1x03, J3 Con1x03, J4 Con1x03, J5 Con1x03, Q1 BC849, U1 TA2003, U2 LM555xM, U3 SSM2211S

Commit message: new DIY version
Parts:
- RV1, RV2: footprint 3Channel-PiezoAmp:RD901F-ALPHA-3D -> Indosluch_AM:RD901F-ALPHA-HandSolder
