File: Indosluch_AM/Indosluch_AM/Indosluch_AM.sch (KiCad schematic (older format))
At the start: 41 parts, among them J1 Con1x03, J2 Con1x03, J3 Con1x03, J4 Con1x03, J5 Con1x03, Q1 BC849, U1 TA2003, U2 LM555xM, U3 SSM2211S

Commit message: new DIY versions
Parts:
- removed C9: 100uF, Capacitor_THT:CP_Radial_D6.3mm_P2.50mm, symbol Device:CP
- added C17: 470nF, BioAmp:C_1206_dusjagr, symbol Device:C
- added C18: 100nF, BioAmp:C_1206_dusjagr, symbol Device:C
- added D1, D2: LED, 3Channel-PiezoAmp:LED_0805_2012Metric_Pad1.15x1.40mm_HandSolder, symbol Device:LED
- added J6: Con1x03, Indosluch_AM:PinHeader_1x03_HandSolder, symbol Connector:Conn_01x03_Female
- added J7: Conn_01x02_Female, Indosluch_AM:PinHeader_1x02_P2.54mm_HandSolder, symbol Connector:Conn_01x02_Female
- added LOGO1: Logo, Indosluch_AM:Indosluch_logos, symbol Connector:Conn_01x01_Female
- added R12, R14: 10K, BioAmp:R_1206_dusjagr, symbol Device:R
- added R13: 330, BioAmp:R_1206_dusjagr, symbol Device:R
- added R15: 0, BioAmp:R_1206_dusjagr, symbol Device:R
- C4: footprint Capacitor_THT:CP_Radial_D6.3mm_P2.50mm -> Indosluch_AM:Capacitor_Radial_D6.3mm_P2.50mm
- C8: value 10uF -> 470uF; footprint Capacitor_THT:CP_Radial_D5.0mm_P2.50mm -> Indosluch_AM:Capacitor_Radial_D6.3mm_P2.50mm
- J1, J2, J3, J4, J5: footprint Connector_PinHeader_2.54mm:PinHeader_1x03_P2.54mm_Vertical -> Indosluch_AM:PinHeader_1x03_HandSolder
- L1: footprint BioAmp:PJ301M-12_dusjagr_3d -> Indosluch_AM:PJ301M-12_dusjagr_handSolder
- Q1: footprint 3Channel-PiezoAmp:SOT-23_Handsoldering -> Indosluch_AM:SOT-23_Handsoldering
- R5: value 470 -> 10K
- RV1, RV2: footprint 3Channel-PiezoAmp:RD901F-ALPHA-3D -> Indosluch_AM:RD901F-ALPHA-HandSolder
- U1: footprint Package_SO:SOP-16_3.9x9.9mm_P1.27mm -> Indosluch_AM:SOP-16_HandSolder
- U2, U3: footprint Package_SO:SOIC-8_3.9x4.9mm_P1.27mm -> Indosluch_AM:SOIC-8_HandSolder
Connections:
- net AM-Filter-OUT: now also C17.2
- net GND: now also U3.1 (SHUTDOWN), U3.7 (V-), C18.1, D1.1 (K), J6.1 (Pin_1), J7.1 (Pin_1), R14.1
- net Speaker+Output: now also C8.1, J5.3 (Pin_3), U3.8 (VoutB), J6.3 (Pin_3); no longer J5.2 (Pin_2)
- net Speaker-Output: now also J5.2 (Pin_2), U3.5 (VoutA), R12.1; no longer J5.3 (Pin_3)
- net VCC: now also U3.6 (V+), D2.2 (A), J7.2 (Pin_2)
- net at C14.2, R8.1, R9.2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: now also R15.1; no longer U2.4 (R)
- net at U3.2 (BYPASS): now also U3.3 (IN+), C18.2
- net at U3.4 (IN-): now also R5.1, R12.2
- net at C8.2: now also J6.2 (Pin_2), R13.2
- net at R5.2: now also C17.1
- new net: R15.2, U2.4 (R)
- new net: D1.2 (A), R13.1
- new net: D2.1 (K), R14.2
Other:
- moved on the sheet: C8, J5
